File: keyboard.sch (KiCad schematic (older format))
At the start: 192 parts, among them SW1 SW_Push, U1 ATmega32U4-AU, Y1 16MHz

Commit message: Reversed stabilizers for spacebars
Parts:
- MX_LSPACE1: footprint MX_Alps_Hybrid:MX-2.75U-NoLED -> MX_Alps_Hybrid:MX-2.75U-ReversedStabilizers-NoLED
- MX_RSPACE1: footprint MX_Alps_Hybrid:MX-2.25U-NoLED -> MX_Alps_Hybrid:MX-2.25U-ReversedStabilizers-NoLED
Changed lines of the file:
@@
 F 0 "MX_RSPACE1" H 17083 5973 60  0000 C CNN
 F 1 "MX-NoLED" H 17083 5899 20  0000 C CNN
-F 2 "MX_Alps_Hybrid:MX-2.25U-NoLED" H 16425 5725 60  0001 C CNN
+F 2 "MX_Alps_Hybrid:MX-2.25U-ReversedStabilizers-NoLED" H 16425 5725 60  0001 C CNN
 F 3 "" H 16425 5725 60  0001 C CNN
 	1    17050 5750
@@
 F 0 "MX_LSPACE1" H 16033 5973 60  0000 C CNN
 F 1 "MX-NoLED" H 16033 5899 20  0000 C CNN
-F 2 "MX_Alps_Hybrid:MX-2.75U-NoLED" H 15375 5725 60  0001 C CNN
+F 2 "MX_Alps_Hybrid:MX-2.75U-ReversedStabilizers-NoLED" H 15375 5725 60  0001 C CNN
 F 3 "" H 15375 5725 60  0001 C CNN
 	1    16000 5750

Commit message: Unknown changes
Parts:
- Y1: footprint Crystal:Crystal_SMD_3225-4Pin_3.2x2.5mm -> Crystal:Crystal_SMD_3225-4Pin_3.2x2.5mm_HandSoldering
Changed lines of the file:
@@
 F 0 "Y1" V 2904 2744 50  0000 L CNN
 F 1 "16MHz" V 2995 2744 50  0000 L CNN
-F 2 "Crystal:Crystal_SMD_3225-4Pin_3.2x2.5mm" H 2950 2600 50  0001 C CNN
+F 2 "Crystal:Crystal_SMD_3225-4Pin_3.2x2.5mm_HandSoldering" H 2950 2600 50  0001 C CNN
 F 3 "~" H 2950 2600 50  0001 C CNN
 	1    2950 2600
